Commit message: Updated irb6700 robot urdfs

File: src/telekinesis_urdfs/models/example-robot-data/robots/abb/irb6700_description/urdf/irb6700_200_260.urdf (robot description, URDF)
Before this commit: robot abb_irb6700_200_260, 12 links, 11 joints
Links:
- removed link cylinder
- removed link piston
Joints:
- removed joint cylinder_joint
- removed joint piston_joint

File: src/telekinesis_urdfs/models/example-robot-data/robots/abb/irb6700_description/urdf/irb6700_235_265.urdf (robot description, URDF)
Before this commit: robot abb_irb6700_235_265, 12 links, 11 joints
Links:
- removed link cylinder
- removed link piston
Joints:
- removed joint cylinder_joint
- removed joint piston_joint
