Commit message: feat: Added hande, rg2, restrytuced folder structures, and added contribuiting.md

File: src/telekinesis_urdfs/models/example-robot-data/robots/universal_robots/urdf/ur5_robotiq_2f_85.urdf (robot description, URDF)
Before this commit: robot ur5, 20 links, 19 joints
Links:
- link robotiq_85_base_link: mass 0.636951 -> 6.6320197e-01; geometry collision mesh filename=package://example-robot-data/tools/robotiq/meshes/collision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; visual mesh filename=package://example-robot-data/tools/robotiq/meshes/visual/2f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
- link robotiq_85_left_finger_link: mass 0.027309 -> 4.260376752e-02; geometry collision mesh filename=package://example-robot-data/tools/robotiq/meshes/collision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; visual mesh filename=package://example-robot-data/tools/robotiq/meshes/visual/2f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
- link robotiq_85_left_finger_tip_link: mass 0.019555 -> 4.268588744e-02; geometry collision mesh filename=package://example-robot-data/tools/robotiq/meshes/collision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; visual mesh filename=package://example-robot-data/tools/robotiq/meshes/visual/2f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
- link robotiq_85_left_inner_knuckle_link: mass 0.029951 -> 2.969376448e-02; geometry collision mesh filename=package://example-robot-data/tools/robotiq/meshes/collision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; visual mesh filename=package://example-robot-data/tools/robotiq/meshes/visual/2f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
- link robotiq_85_left_knuckle_link: mass 0.018491 -> 1.384773208e-02; geometry collision mesh filename=package://example-robot-data/tools/robotiq/meshes/collision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; visual mesh filename=package://example-robot-data/tools/robotiq/meshes/visual/2f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
- link robotiq_85_right_finger_link: mass 0.027309 -> 4.260376752000000e-02; geometry collision mesh filename=package://example-robot-data/tools/robotiq/meshes/collision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; visual mesh filename=package://example-robot-data/tools/robotiq/meshes/visual/2f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
- link robotiq_85_right_finger_tip_link: mass 0.019555 -> 4.268588744e-02; geometry collision mesh filename=package://example-robot-data/tools/robotiq/meshes/collision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; visual mesh filename=package://example-robot-data/tools/robotiq/meshes/visual/2f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
- link robotiq_85_right_inner_knuckle_link: mass 0.029951 -> 2.969376448e-02; geometry collision mesh filename=package://example-robot-data/tools/robotiq/meshes/collision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; visual mesh filename=package://example-robot-data/tools/robotiq/meshes/visual/2f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
- link robotiq_85_right_knuckle_link: mass 0.018491 -> 1.384773208e-02; geometry collision mesh filename=package://example-robot-data/tools/robotiq/meshes/collision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; visual mesh filename=package://example-robot-data/tools/robotiq/meshes/visual/2f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
Joints:
- joint robotiq_85_left_finger_joint: origin xyz=-0.00408552455 -0.03148604435 0.0 rpy=0 0 0 -> xyz=0.03152616 0.0 -0.00376347 rpy=0 0 0
- joint robotiq_85_left_finger_tip_joint: axis 0 0 1 -> 0 -1 0; limit lower=-3.14 upper=3.14 effort=0.1 velocity=3.14 -> (none); origin xyz=0.04303959807 -0.03759940821 0.0 rpy=0.0 0.0 0.0 -> xyz=0.00563134 0.0 0.04718515 rpy=0 0 0; parent robotiq_85_left_inner_knuckle_link -> robotiq_85_left_finger_link; type revolute -> continuous
- joint robotiq_85_left_inner_knuckle_joint: axis 0 0 1 -> 0 -1 0; limit lower=-3.14 upper=3.14 effort=0.1 velocity=3.14 -> (none); mimic joint=robotiq_85_left_knuckle_joint offset=0 -> joint=robotiq_85_left_knuckle_joint; origin xyz=0.06142 0.0127 0 rpy=3.14 0.0 0.0 -> xyz=0.0127 0.0 0.06142 rpy=0 0 0; type revolute -> continuous
- joint robotiq_85_left_knuckle_joint: axis 0 0 1 -> 0 -1 0; limit lower=0.0 upper=0.80285 effort=1000 velocity=3.14 -> lower=0.0 upper=0.8 effort=50 velocity=0.5; origin xyz=0.05490451627 0.03060114443 0.0 rpy=3.14 0.0 0.0 -> xyz=0.03060114 0.0 0.05490452 rpy=0 0 0
- joint robotiq_85_right_finger_joint: origin xyz=-0.00408552455 -0.03148604435 0.0 rpy=0 0 0 -> xyz=-0.03152616 0.0 -0.00376347 rpy=0 0 0
- joint robotiq_85_right_finger_tip_joint: axis 0 0 1 -> 0 -1 0; limit lower=-3.14 upper=3.14 effort=0.1 velocity=3.14 -> (none); mimic joint=robotiq_85_left_knuckle_joint multiplier=-1 -> joint=robotiq_85_left_knuckle_joint; origin xyz=0.04303959807 -0.03759940821  0.0 rpy=0.0 0.0 0.0 -> xyz=-0.00563134 0.0 0.04718515 rpy=0 0 0; parent robotiq_85_right_inner_knuckle_link -> robotiq_85_right_finger_link; type revolute -> continuous
- joint robotiq_85_right_inner_knuckle_joint: axis 0 0 1 -> 0 -1 0; limit lower=-3.14 upper=3.14 effort=0.1 velocity=3.14 -> (none); mimic joint=robotiq_85_left_knuckle_joint offset=0 -> joint=robotiq_85_left_knuckle_joint multiplier=-1; origin xyz=0.06142 -0.0127 0 rpy=0 0 0 -> xyz=-0.0127 0.0 0.06142 rpy=0 0 0; type revolute -> continuous
- joint robotiq_85_right_knuckle_joint: axis 0 0 1 -> 0 -1 0; limit lower=-3.14 upper=3.14 effort=1000 velocity=3.14 -> lower=-0.8 upper=0.0 effort=50 velocity=0.5; mimic joint=robotiq_85_left_knuckle_joint -> joint=robotiq_85_left_knuckle_joint multiplier=-1; origin xyz=0.05490451627 -0.03060114443 0.0 rpy=0.0 0.0 0.0 -> xyz=-0.03060114 0.0 0.05490452 rpy=0 0 0
