Commit message: fix: Piab urdf updated with glb visual mesh. Moved glb and fbx inside piab/meshes/visual/

File: src/telekinesis_urdfs/models/example-robot-data/tools/piab/urdf/picobot_electric.urdf (robot description, URDF)
Before this commit: robot piab_picobot_electric, 2 links, 1 joints
Links:
- link picobot_electric_base_link: geometry collision mesh filename=package://example-robot-data/tools/piab/meshes/collision/pi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; visual mesh filename=package://example-robot-data/tools/piab/meshes/visual/piCOB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
