Commit message: Updated velocity for rg2

File: src/telekinesis_urdfs/models/example-robot-data/tools/onrobot/urdf/onrobot_rg2_model.urdf (robot description, URDF)
Before this commit: robot onrobot_rg2_model, 8 links, 7 joints
Joints:
- joint finger_joint: limit lower=-0.558505 upper=0.785398 effort=1000 velocity=100.0 -> lower=-0.558505 upper=0.785398 effort=1000 velocity=2.0
- joint left_inner_finger_joint: limit lower=-0.872665 upper=0.872665 effort=1000 velocity=100.0 -> lower=-0.872665 upper=0.872665 effort=1000 velocity=2.0
- joint left_inner_knuckle_joint: limit lower=-0.785398 upper=0.785398 effort=1000 velocity=100.0 -> lower=-0.785398 upper=0.785398 effort=1000 velocity=2.0
- joint right_inner_finger_joint: limit lower=-0.872665 upper=0.872665 effort=1000 velocity=100.0 -> lower=-0.872665 upper=0.872665 effort=1000 velocity=2.0
- joint right_inner_knuckle_joint: limit lower=-0.785398 upper=0.785398 effort=1000 velocity=100.0 -> lower=-0.785398 upper=0.785398 effort=1000 velocity=2.0
- joint right_outer_knuckle_joint: limit lower=-0.785398 upper=0.785398 effort=1000 velocity=100.0 -> lower=-0.785398 upper=0.785398 effort=1000 velocity=2.0

Commit message: Updated rg urdfs

File: src/telekinesis_urdfs/models/example-robot-data/tools/onrobot/urdf/onrobot_rg2_model.urdf (robot description, URDF)
Before this commit: robot onrobot_rg2_model, 8 links, 7 joints
Joints:
- joint finger_joint: limit lower=-0.558505 upper=0.785398 effort=1000 velocity=2.0 -> lower=-0.558505 upper=0.785398 effort=50 velocity=2.0
- joint left_inner_finger_joint: limit lower=-0.872665 upper=0.872665 effort=1000 velocity=2.0 -> lower=-0.872665 upper=0.872665 effort=50 velocity=2.0
- joint left_inner_knuckle_joint: limit lower=-0.785398 upper=0.785398 effort=1000 velocity=2.0 -> lower=-0.785398 upper=0.785398 effort=50 velocity=2.0
- joint right_inner_finger_joint: limit lower=-0.872665 upper=0.872665 effort=1000 velocity=2.0 -> lower=-0.872665 upper=0.872665 effort=50 velocity=2.0
- joint right_inner_knuckle_joint: limit lower=-0.785398 upper=0.785398 effort=1000 velocity=2.0 -> lower=-0.785398 upper=0.785398 effort=50 velocity=2.0
- joint right_outer_knuckle_joint: limit lower=-0.785398 upper=0.785398 effort=1000 velocity=2.0 -> lower=-0.785398 upper=0.785398 effort=50 velocity=2.0

File: src/telekinesis_urdfs/models/example-robot-data/tools/onrobot/urdf/onrobot_rg6_model.urdf (robot description, URDF)
Before this commit: robot onrobot_rg6_model, 8 links, 7 joints
Joints:
- joint finger_joint: limit lower=-0.628319 upper=0.628319 effort=1000 velocity=2.0 -> lower=-0.628319 upper=0.628319 effort=50 velocity=2.0
- joint left_inner_finger_joint: limit lower=-0.872665 upper=0.872665 effort=1000 velocity=2.0 -> lower=-0.872665 upper=0.872665 effort=50 velocity=2.0
- joint left_inner_knuckle_joint: limit lower=-0.628319 upper=0.628319 effort=1000 velocity=2.0 -> lower=-0.628319 upper=0.628319 effort=50 velocity=2.0
- joint right_inner_finger_joint: limit lower=-0.872665 upper=0.872665 effort=1000 velocity=2.0 -> lower=-0.872665 upper=0.872665 effort=50 velocity=2.0
- joint right_inner_knuckle_joint: limit lower=-0.628319 upper=0.628319 effort=1000 velocity=2.0 -> lower=-0.628319 upper=0.628319 effort=50 velocity=2.0
- joint right_outer_knuckle_joint: limit lower=-0.628319 upper=0.628319 effort=1000 velocity=2.0 -> lower=-0.628319 upper=0.628319 effort=50 velocity=2.0
